File: Term24.kicad_sch (KiCad schematic)
At the start: 53 parts, among them J1 USB_B, J11 VGA DE15, J14 Conn_01x06, J15 Conn_01x06, J3 DE9_Plug, J5 Mini-DIN-6, J6 Conn_01x08, J7 AudioJack3, SW1 SW_DIP_x02, SW11 SW_Push, SW2 SW_DIP_x02, SW3 SW_SPDT, U1 PIC24EP512GP202-I/SP, U5 LM1117T-3.3

Commit message: Add files via upload
Parts:
- removed C24: C_Polarized_Small_US, Capacitor_THT:CP_Radial_D6.3mm_P2.50mm, symbol Device:C_Polarized_Small_US
- removed J3: DE9_Plug, Connector_Dsub:DSUB-9_Pins_Vertical_P2.77x2.84mm_MountingHoles, symbol Connector:DE9_Plug
- removed J6: Conn_01x08, Connector_PinSocket_2.54mm:PinSocket_1x08_P2.54mm_Horizontal, symbol Connector_Generic:Conn_01x08
- removed J7: AudioJack3, Connector_Audio:Jack_3.5mm_CUI_SJ1-3535NG_Horizontal_CircularHoles, symbol Connector:AudioJack3
- removed R21, R22, R23, R24, R25, R26, R27, R4, R5, R6: R_US, Resistor_THT:R_Axial_DIN0207_L6.3mm_D2.5mm_P10.16mm_Horizontal, symbol Device:R_US
- removed SW1: SW_DIP_x02, Button_Switch_THT:SW_DIP_SPSTx02_Slide_9.78x7.26mm_W7.62mm_P2.54mm, symbol Switch:SW_DIP_x02
- removed SW2: SW_DIP_x02, Button_Switch_THT:SW_DIP_SPSTx02_Piano_10.8x6.64mm_W7.62mm_P2.54mm, symbol Switch:SW_DIP_x02
- added J2: Conn_01x16, Connector_PinSocket_2.54mm:PinSocket_1x16_P2.54mm_Horizontal, symbol Connector_Generic:Conn_01x16
- added JP1, JP10, JP11, JP12, JP2, JP3, JP4, JP5, JP6, JP7, JP8, JP9: Jumper_2_Open, Jumper:SolderJumper-2_P1.3mm_Open_Pad1.0x1.5mm, symbol Jumper:Jumper_2_Open
- added R33, R34, R35, R37, R38, R39, R40, R41, R42, R43, R44, R45, R46: R_US, Resistor_THT:R_Axial_DIN0207_L6.3mm_D2.5mm_P10.16mm_Horizontal, symbol Device:R_US
- added SW10: SW_DIP_x04, Button_Switch_THT:SW_DIP_SPSTx04_Slide_9.78x12.34mm_W7.62mm_P2.54mm, symbol Switch:SW_DIP_x04
- added SW4, SW5, SW6, SW7, SW8, SW9: SW_Push, Button_Switch_THT:SW_PUSH_6mm_H7.3mm, symbol Switch:SW_Push
- added TP1, TP10, TP100, TP101, TP102, TP103, TP104, TP105, TP106, TP107, TP108, TP109, TP11, TP110, TP111, TP112, TP113, TP114, TP115, TP116, TP117, TP118, TP119, TP12, TP120, TP121, TP122, TP123, TP124, TP125, TP126, TP127, TP128, TP129, TP13, TP130, TP131, TP132, TP133, TP134, TP135, TP136, TP137, TP138, TP139, TP14, TP140, TP141, TP142, TP143, TP144, TP145, TP146, TP147, TP148, TP15, TP16, TP17, TP18, TP19, TP20, TP21, TP22, TP23, TP24, TP25, TP26, TP27, TP28, TP29, TP30, TP31, TP32, TP33, TP34, TP35, TP36, TP37, TP38, TP39, TP40, TP41, TP42, TP43, TP44, TP45, TP46, TP47, TP48, TP49, TP50, TP51, TP52, TP53, TP54, TP55, TP56, TP57, TP58, TP59, TP6, TP60, TP61, TP62, TP63, TP64, TP65, TP66, TP67, TP68, TP69, TP7, TP70, TP71, TP72, TP73, TP74, TP75, TP76, TP77, TP78, TP79, TP8, TP80, TP81, TP82, TP83, TP84, TP85, TP86, TP87, TP88, TP89, TP9, TP90, TP91, TP92, TP93, TP94, TP95, TP96, TP97, TP98, TP99: TestPoint, Hardware:PinHeader_1x01_P2.54mm_Vertical_TestPoint, symbol Connector:TestPoint
- R36: Field4 20K -> (none)
Connections:
- net AUDIO-D is gone; now on net PORT-A0-3V3: U1.2 (AN0/OA2OUT/RA0)
- net OPTION-A is gone; now on net ICSP-CLK: U1.5 (PGEC3/VREF+/AN3/OA1OUT/RPI33/CTED1/RB1)
- net OPTION-B is gone; now on net ICSP-DAT: U1.4 (PGED3/VREF-/AN2/C2IN1-/*SS1/RPI32/CTED2/RB0)
- net +3V3: now also J2.12 (Pin_12)
- net +5V: now also J2.11 (Pin_11)
- net GND: now also J2.13 (Pin_13), J2.14 (Pin_14), R33.1, R34.1, R38.2, R40.2, R42.2, R44.2, R46.2, SW4.2, SW5.2, SW6.2, SW7.2, SW8.2, SW9.2
- net ICSP-CLK: now also SW10.3; no longer U1.6 (PGEC1/AN4/C1IN1+/RPI34/RB2)
- net ICSP-DAT: now also SW10.4; no longer U1.7 (PGED1/AN5/C1IN1-/RP35/RB3)
- net ~{MCLR}: now also J2.10 (Pin_10)
- net JOY-A: now reaches RN1.2 (R1)
- net JOY-A: now also A1.22 (D7), JP12.1 (A), SW8.1
- net PORT-A0-3V3: now reaches R36.1
- net PORT-A0-3V3: now also JP1.2 (B), JP7.2 (B), R35.2
- net UNO-RX: now reaches A1.15 (D0/RX)
- net UNO-RX: now also SW10.8
- net UNO-TX: now reaches A1.16 (D1/TX)
- net UNO-TX: now also SW10.7
- net AUDIO-A renamed PORT-A3-3V3
- net PORT-A3-3V3: now also JP10.2 (B), JP4.2 (B), R41.2, R42.1
- net AUDIO-B renamed PORT-A2-3V3
- net PORT-A2-3V3: now also JP3.2 (B), JP9.2 (B), R39.2, R40.1
- net AUDIO-C renamed PORT-A1-3V3
- net PORT-A1-3V3: now also JP2.2 (B), JP8.2 (B), R37.2, R38.1
- net JOY-BUTTON1 renamed JOY-D
- net JOY-D: now also A1.19 (D4), JP9.1 (A), SW5.1; no longer A1.18 (D3)
- net JOY-BUTTON2 renamed JOY-R
- net JOY-R: now also RN1.7 (R6), JP7.1 (A), SW7.1; no longer RN1.4 (R3)
- net JOY-DOWN renamed JOY-B
- net JOY-B: now also RN1.3 (R2), JP11.1 (A), SW9.1; no longer RN1.8 (R7)
- net JOY-LEFT renamed JOY-U
- net JOY-U: now also RN1.4 (R3), JP10.1 (A), SW4.1; no longer RN1.7 (R6)
- net JOY-RIGHT renamed JOY-L
- net JOY-L: now also A1.18 (D3), JP8.1 (A), SW6.1; no longer A1.19 (D4)
- net JOY-SELECT: no longer names the net of A1.23 (D8)
- net JOY-SELECT: no longer RN1.3 (R2)
- net JOY-UP renamed SERIAL-CLK-TX
- net SERIAL-CLK-TX: now also A1.28 (D13), J15.5 (Pin_5), J5.5, U1.15 (PGEC2/ASCL2/RP38/RB6^), J2.1 (Pin_1), SW10.1; no longer A1.22 (D7)
- removed net SERIAL-CLK-TX-SCL: A1.14 (SCL/A5), A1.28 (D13), A1.32 (SCL/A5), J15.5 (Pin_5), J5.5, U1.15 (PGEC2/ASCL2/RP38/RB6^)
- net SERIAL-MISO renamed SERIAL-MISO-EX
- net SERIAL-MISO-EX: now also J2.3 (Pin_3)
- net SERIAL-MOSI-RX-SDA renamed SERIAL-MOSI-RX
- net SERIAL-MOSI-RX: now also RN1.8 (R7), J2.2 (Pin_2), SW10.2; no longer A1.13 (SDA/A4), A1.31 (SDA/A4)
- new net: R34.2, SW10.5
- new net: R33.2, SW10.6
- new net PORT-A0-5V: J2.9 (Pin_9), JP1.1 (A), R35.1
- new net PORT-A1-5V: J2.8 (Pin_8), JP2.1 (A), R37.1
- new net PORT-A2-5V: J2.7 (Pin_7), JP3.1 (A), R39.1
- new net PORT-A3-5V: J2.6 (Pin_6), JP4.1 (A), R41.1
- new net PORT-B2-3V3: JP11.2 (B), JP5.2 (B), R43.2, R44.1, U1.6 (PGEC1/AN4/C1IN1+/RPI34/RB2)
- new net PORT-B2-5V: J2.5 (Pin_5), JP5.1 (A), R43.1
- new net PORT-B3-3V3: JP12.2 (B), JP6.2 (B), R45.2, R46.1, U1.7 (PGED1/AN5/C1IN1-/RP35/RB3)
- new net PORT-B3-5V: J2.4 (Pin_4), JP6.1 (A), R45.1
- no-connect marks 25 -> 175
Other:
- note added: "1.1K then 2.2K to drop 5V to 3V3"
- note added: "10K ohms"
- note added: "Steven Chad Burrow, July 2026"
- note added: "Term24"

Commit message: Add files via upload
Parts:
- added C3: C_Polarized_US, Capacitor_THT:CP_Radial_D8.0mm_P3.50mm, symbol Device:C_Polarized_US
- added JP13: Jumper_2_Open, Jumper:SolderJumper-2_P1.3mm_Open_Pad1.0x1.5mm, symbol Jumper:Jumper_2_Open
Connections:
- net +3V3: now also C3.1, JP13.2 (B)
- net GND: now also C3.2
- net UNO-3V3: now reaches A1.4 (3V3)
- net UNO-3V3: now also JP13.1 (A)
- no-connect marks 175 -> 174
